File: Adapter-VCNL4010.kicad_pcb (KiCad board)
At the start: 2 copper layers, 13.5 x 11 mm, 8 parts, among them J1 Conn_01x03, J2 Conn_01x03, U1 VCNL4010

Commit message: added PDF
Other:
- board text added: "GND"
- board text added: "INT"
- board text added: "SCLK"
- board text added: "SDAT"
- board text added: "VCC"
- board text added: "VCC_LED"
