File: Adapter-VCNL4010.sch (KiCad schematic (older format))
At the start: 11 parts, among them J1 Conn_01x04, J2 Conn_01x04

Commit message: Created gerbers
Parts:
- removed R1, R2, R3: TBD, Resistor_SMD:R_0805_2012Metric_Pad1.20x1.40mm_HandSolder, symbol Device:R_Small
- J1, J2: value Conn_01x04 -> Conn_01x03; footprint Connector_PinHeader_2.54mm:PinHeader_1x04_P2.54mm_Vertical -> Connector_PinHeader_2.54mm:PinHeader_1x03_P2.54mm_Vertical; symbol Connector_Generic:Conn_01x04 -> Connector_Generic:Conn_01x03
- U1: renamed from U?; footprint (none) -> ak:VCNL4010_HS
- gave numbers to parts that had none: 3
Connections:
- net labels added: VCC, VCC_LED
- wire segments 35 -> 31
Changed lines of the file:
@@
 Wire Wire Line
 	5550 4250 5550 4200
-$Comp
-L Device:R_Small R1
-U 1 1 619C402F
-P 7050 2950
-F 0 "R1" H 6991 2996 50  0000 R CNN
-F 1 "TBD" H 6991 2905 50  0000 R CNN
-F 2 "Resistor_SMD:R_0805_2012Metric_Pad1.20x1.40mm_HandSolder" H 7050 2950 50  0001 C CNN
-F 3 "~" H 7050 2950 50  0001 C CNN
-	1    7050 2950
-	-1   0    0    -1
-$EndComp
-$Comp
-L Device:R_Small R2
-U 1 1 619C44B1
-P 6750 2950
-F 0 "R2" H 6691 2996 50  0000 R CNN
-F 1 "TBD" H 6691 2905 50  0000 R CNN
-F 2 "Resistor_SMD:R_0805_2012Metric_Pad1.20x1.40mm_HandSolder" H 6750 2950 50  0001 C CNN
-F 3 "~" H 6750 2950 50  0001 C CNN
-	1    6750 2950
-	-1   0    0    -1
-$EndComp
-$Comp
-L Device:R_Small R3
-U 1 1 619C4680
-P 6450 2950
-F 0 "R3" H 6391 2996 50  0000 R CNN
-F 1 "TBD" H 6391 2905 50  0000 R CNN
-F 2 "Resistor_SMD:R_0805_2012Metric_Pad1.20x1.40mm_HandSolder" H 6450 2950 50  0001 C CNN
-F 3 "~" H 6450 2950 50  0001 C CNN
-	1    6450 2950
-	-1   0    0    -1
-$EndComp
-Wire Wire Line
-	6750 2800 6750 2850
-Wire Wire Line
-	7050 2800 7050 2850
 Wire Wire Line
 	4650 2950 4650 2900
@@
 Wire Wire Line
 	4650 2900 5000 2900
-Text Label 7450 3400 2    50   ~ 0
+Text Label 6500 3400 2    50   ~ 0
 SCLK
-Text Label 7450 3500 2    50   ~ 0
+Text Label 6500 3500 2    50   ~ 0
 SDAT
-Text Label 7450 3200 2    50   ~ 0
+Text Label 6500 3200 2    50   ~ 0
 INT
-$Comp
-L Connector_Generic:Conn_01x04 J1
-U 1 1 619CC655
-P 2150 5150
-F 0 "J1" H 2150 5350 50  0000 C CNN
-F 1 "Conn_01x04" H 2068 5376 50  0001 C CNN
-F 2 "Connector_PinHeader_2.54mm:PinHeader_1x04_P2.54mm_Vertical" H 2150 5150 50  0001 C CNN
-F 3 "~" H 2150 5150 50  0001 C CNN
-	1    2150 5150
-	-1   0    0    -1
-$EndComp
-$Comp
-L Connector_Generic:Conn_01x04 J2
-U 1 1 619CF6B4
-P 4050 5150
-F 0 "J2" H 4000 5350 50  0000 L CNN
-F 1 "Conn_01x04" H 4130 5051 50  0001 L CNN
-F 2 "Connector_PinHeader_2.54mm:PinHeader_1x04_P2.54mm_Vertical" H 4050 5150 50  0001 C CNN
-F 3 "~" H 4050 5150 50  0001 C CNN
-	1    4050 5150
-	1    0    0    -1
-$EndComp
 Wire Notes Line
-	2000 4500 4350 4500
+	4750 4750 6500 4750
 Wire Notes Line
-	4350 4500 4350 5650
+	6500 4750 6500 5900
 Wire Notes Line
-	4350 5650 2000 5650
+	6500 5900 4750 5900
 Wire Notes Line
-	2000 5650 2000 4500
-Text Notes 2150 4650 0    79   ~ 0
+	4750 5900 4750 4750
+Text Notes 4900 4900 0    79   ~ 0
 Breadboard Pinheader
 $Comp
-L ak:VCNL4010 U?
+L ak:VCNL4010 U1
 U 1 1 619BBC1A
 P 5550 2900
-F 0 "U?" H 5150 3200 50  0000 C CNN
+F 0 "U1" H 5150 3200 50  0000 C CNN
 F 1 "VCNL4010" H 5850 1700 50  0000 C CNN
-F 2 "" H 5050 3400 50  0001 C CNN
+F 2 "ak:VCNL4010_HS" H 5050 3400 50  0001 C CNN
 F 3 "" H 5050 3400 50  0001 C CNN
 	1    5550 2900
 	1    0    0    -1
 $EndComp
-Wire Wire Line
-	6100 3200 6450 3200
-Wire Wire Line
-	6450 3050 6450 3200
-Connection ~ 6450 3200
-Wire Wire Line
-	6450 3200 7450 3200
-Wire Wire Line
-	6450 2850 6450 2800
-Wire Wire Line
-	6450 2800 6750 2800
-Connection ~ 6750 2800
-Wire Wire Line
-	6750 2800 7050 2800
 Wire Wire Line
 	5550 4200 5500 4200
@@
 	4300 2900 4650 2900
 $Comp
-L Device:R_Small R?
+L Device:R_Small R4
 U 1 1 619CA19C
 P 4050 2900
-F 0 "R?" V 4246 2900 50  0000 C CNN
+F 0 "R4" V 4246 2900 50  0000 C CNN
 F 1 "10R" V 4155 2900 50  0000 C CNN
 F 2 "Resistor_SMD:R_0805_2012Metric_Pad1.20x1.40mm_HandSolder" H 4050 2900 50  0001 C CNN
@@
 	3950 2900 3750 2900
 $Comp
-L Device:C_Small C?
+L Device:C_Small C4
 U 1 1 619CD0D5
 P 4650 2500
-F 0 "C?" H 4742 2546 50  0000 L CNN
+F 0 "C4" H 4742 2546 50  0000 L CNN
 F 1 "100nF" H 4742 2455 50  0000 L CNN
 F 2 "Capacitor_SMD:C_0805_2012Metric_Pad1.18x1.45mm_HandSolder" H 4650 2500 50  0001 C CNN
@@
 $EndComp
 $Comp
-L power:GND #PWR?
+L power:GND #PWR0104
 U 1 1 619CD0DB
 P 4650 2650
-F 0 "#PWR?" H 4650 2400 50  0001 C CNN
+F 0 "#PWR0104" H 4650 2400 50  0001 C CNN
 F 1 "GND" H 4655 2477 50  0001 C CNN
 F 2 "" H 4650 2650 50  0001 C CNN
@@
 	4650 2650 4650 2600
 $Comp
-L Device:C_Small C?
+L Device:C_Small C3
 U 1 1 619CD0E2
 P 4300 2500
-F 0 "C?" H 4392 2546 50  0000 L CNN
+F 0 "C3" H 4392 2546 50  0000 L CNN
 F 1 "22uF" H 4392 2455 50  0000 L CNN
 F 2 "Capacitor_SMD:C_0805_2012Metric_Pad1.18x1.45mm_HandSolder" H 4300 2500 50  0001 C CNN
@@
 $EndComp
 $Comp
-L power:GND #PWR?
+L power:GND #PWR0105
 U 1 1 619CD0E8
 P 4300 2650
-F 0 "#PWR?" H 4300 2400 50  0001 C CNN
+F 0 "#PWR0105" H 4300 2400 50  0001 C CNN
 F 1 "GND" H 4305 2477 50  0001 C CNN
 F 2 "" H 4300 2650 50  0001 C CNN
@@
 Wire Wire Line
 	4650 2350 5550 2350
-Wire Wire Line
-	6100 3500 7050 3500
-Wire Wire Line
-	6100 3400 6750 3400
-Wire Wire Line
-	6750 3050 6750 3400
-Connection ~ 6750 3400
-Wire Wire Line
-	6750 3400 7450 3400
-Wire Wire Line
-	7050 3050 7050 3500
-Connection ~ 7050 3500
-Wire Wire Line
-	7050 3500 7450 3500
 NoConn ~ 5000 3700
 NoConn ~ 5000 3800
+Text Label 3750 2350 0    50   ~ 0
+VCC_LED
+Text Label 3750 2900 0    50   ~ 0
+VCC
+Wire Wire Line
+	5100 5300 5500 5300
+Wire Wire Line
+	5100 5400 5500 5400
+Wire Wire Line
+	5500 5500 5100 5500
+Wire Wire Line
+	5750 5300 6000 5300
+Wire Wire Line
+	5750 5400 6000 5400
+Wire Wire Line
+	6000 5500 5950 5500
+Wire Wire Line
+	6100 3200 6500 3200
+Wire Wire Line
+	6100 3400 6500 3400
+Wire Wire Line
+	6100 3500 6500 3500
+$Comp
+L Connector_Generic:Conn_01x03 J2
+U 1 1 619CF6B4
+P 6200 5400
+F 0 "J2" H 6150 5600 50  0000 L CNN
+F 1 "Conn_01x03" H 6280 5301 50  0001 L CNN
+F 2 "Connector_PinHeader_2.54mm:PinHeader_1x03_P2.54mm_Vertical" H 6200 5400 50  0001 C CNN
+F 3 "~" H 6200 5400 50  0001 C CNN
+	1    6200 5400
+	1    0    0    -1
+$EndComp
+$Comp
+L Connector_Generic:Conn_01x03 J1
+U 1 1 619CC655
+P 4900 5400
+F 0 "J1" H 4900 5600 50  0000 C CNN
+F 1 "Conn_01x03" H 4818 5626 50  0001 C CNN
+F 2 "Connector_PinHeader_2.54mm:PinHeader_1x03_P2.54mm_Vertical" H 4900 5400 50  0001 C CNN
+F 3 "~" H 4900 5400 50  0001 C CNN
+	1    4900 5400
+	-1   0    0    -1
+$EndComp
+Text Label 5750 5300 0    50   ~ 0
+VCC
+Text Label 5500 5300 2    50   ~ 0
+VCC_LED
+Text Label 5750 5400 0    50   ~ 0
+INT
+Text Label 5500 5500 2    50   ~ 0
+SCLK
+Text Label 5500 5400 2    50   ~ 0
+SDAT
+$Comp
+L power:GND #PWR0106
+U 1 1 619CE030
+P 5950 5550
+F 0 "#PWR0106" H 5950 5300 50  0001 C CNN
+F 1 "GND" H 5955 5377 50  0001 C CNN
+F 2 "" H 5950 5550 50  0001 C CNN
+F 3 "" H 5950 5550 50  0001 C CNN
+	1    5950 5550
+	1    0    0    -1
+$EndComp
+Wire Wire Line
+	5950 5500 5950 5550
 $EndSCHEMATC

Commit message: added PDF
Other:
- moved on the sheet: C1, C2, C3, C4, J1, J2, R4, U1
